Commit message: update

File: xacro/tracer/platform.xacro (robot description, xacro)
@@ -31,3 +31,10 @@
         </actuator>
     </transmission>
+    <gazebo>
+        <plugin name="gazebo_ros_control" filename="libgazebo_ros_control.so">
+            <robotNamespace>/tracer</robotNamespace>
+            <robotParam>/robot_description</robotParam>
+            <legacyModeNS>true</legacyModeNS>
+        </plugin>
+    </gazebo>
 </robot>

File: xacro/tracer/spheres.xacro (robot description, xacro)
@@ -21,4 +21,14 @@
             <axis xyz="1 1 1" />
         </joint>
+        <transmission name="${sphere_name}2chasis_trans">
+            <type>transmission_interface/SimpleTransmission</type>
+            <joint name="${sphere_name}2chasis">
+                <hardwareInterface>EffortJointInterface</hardwareInterface>
+            </joint>
+            <actuator name="${sphere_name}2chasis_motor">
+                <mechanicalReduction>1.0</mechanicalReduction>
+                <hardwareInterface>EffortJointInterface</hardwareInterface>
+            </actuator>
+        </transmission>
     </xacro:macro>
     <xacro:sphere_func sphere_name="front" flag = "1"/>

File: xacro/tracer/tracer.xacro (robot description, xacro)
@@ -1,3 +1,23 @@
 <robot xmlns:xacro="http://www.ros.org/wiki/xacro" name="tracer">
+    <xacro:property name="chasis_radius" value="0.4"/>
+    <xacro:property name="chasis_length" value="0.4"/>
+    <xacro:property name="chasis_mass" value="10.0"/>
+    <xacro:property name="wheel_radius" value="0.12"/>
+    <xacro:property name="wheel_length" value="0.05"/>
+    <xacro:property name="wheel_dist" value="0.6"/>
+    <xacro:property name="wheel_mass" value="10.0"/>
+    <xacro:property name="sphere_radius" value="0.025"/>
+    <xacro:property name="sphere_mass" value="0.1"/>
+    <xacro:property name="lidar_radius" value="0.1"/>
+    <xacro:property name="lidar_length" value="0.1"/>
+    <xacro:property name="lidar_mass" value="0.1"/>
+    <xacro:property name="camera_size_x" value="0.05"/>
+    <xacro:property name="camera_size_y" value="0.2"/>
+    <xacro:property name="camera_size_z" value="0.1"/>
+    <xacro:property name="camera_mass" value="0.1"/>
+    <xacro:property name="imu_l" value="0.05"/>
+    <xacro:property name="imu_w" value="0.05"/>
+    <xacro:property name="imu_h" value="0.01"/>
+    <xacro:property name="imu_m" value="0.5"/>
     <link name="base_link">
         <visual>
@@ -7,7 +27,6 @@
         </visual>
     </link>
-    <xacro:include filename="$(find test_mycar)/xacro/tracer/params.xacro"/>
     <xacro:include filename="$(find test_mycar)/xacro/inertia.xacro"/>
-    <!-- <xacro:include filename="$(find test_mycar)/xacro/tracer/platform.xacro"/> -->
+    <xacro:include filename="$(find test_mycar)/xacro/tracer/platform.xacro"/>
     <xacro:include filename="$(find test_mycar)/xacro/tracer/chasis.xacro"/>
     <xacro:include filename="$(find test_mycar)/xacro/tracer/lidar.xacro"/>
@@ -16,3 +35,4 @@
     <xacro:include filename="$(find test_mycar)/xacro/tracer/spheres.xacro"/>
     <xacro:include filename="$(find test_mycar)/xacro/tracer/wheels.xacro"/>
+    <xacro:include filename="$(find test_mycar)/xacro/tracer/imu.xacro"/>
 </robot>

File: xacro/tracer/wheels.xacro (robot description, xacro)
@@ -38,26 +38,24 @@
     <gazebo>
         <plugin name="differential_drive_controller" filename="libgazebo_ros_diff_drive.so">
-            <!-- <publishWheelTF>true</publishWheelTF> -->
+            <rosDebugLevel>Debug</rosDebugLevel>
+            <publishWheelTF>false</publishWheelTF>
             <robotNamespace>/</robotNamespace>
-            <!-- <publishTf>1</publishTf> -->
-            <publishWheelJointState>true</publishWheelJointState>
+            <publishTf>1</publishTf>
+            <publishWheelJointState>false</publishWheelJointState>
             <alwaysOn>true</alwaysOn>
             <updateRate>100.0</updateRate>
-            <!-- <legacyMode>true</legacyMode> -->
+            <legacyMode>true</legacyMode>
             <leftJoint>left2chasis</leftJoint> <!-- 左轮 -->
             <rightJoint>right2chasis</rightJoint> <!-- 右轮 -->
-            <wheelSeparation>${wheel_dist+wheel_length}</wheelSeparation> <!-- 车轮间距 -->
+            <wheelSeparation>${0.6+wheel_length}</wheelSeparation> <!-- 车轮间距 -->
             <wheelDiameter>${wheel_radius*2}</wheelDiameter> <!-- 车轮直径 -->
-            <!-- <broadcastTF>1</broadcastTF> -->
+            <broadcastTF>1</broadcastTF>
             <wheelTorque>30</wheelTorque>
-            <!-- <wheelAcceleration>1.8</wheelAcceleration> -->
-            <commandTopic>/cmd_vel</commandTopic> <!-- 运动控制话题 -->
+            <wheelAcceleration>1.8</wheelAcceleration>
+            <commandTopic>tracer/cmd_vel</commandTopic> <!-- 运动控制话题 -->
             <odometryFrame>/odom</odometryFrame>
             <odometryTopic>/odom</odometryTopic> <!-- 里程计话题 -->
             <robotBaseFrame>/base_link</robotBaseFrame> <!-- 根坐标系 -->
         </plugin>
-        <!-- <plugin name="gazebo_ros_control" filename="libgazebo_ros_control.so">
-            <robotNamespace>/tracer</robotNamespace>
-        </plugin> -->
     </gazebo>
 </robot>
