Commit message: update

File: xacro/ackermann/front_wheels.xacro (robot description, xacro)
@@ -23,5 +23,5 @@
             <child link="${name}_steering"/>
             <axis xyz="0 0 1"/>
-            <limit lower="-1.0" upper="1.0" velocity="1.0" effort="1000.0"/>
+            <limit lower="-1.52" upper="1.52" velocity="1.0" effort="1000.0"/>
             <origin xyz="${chasis_l/2-wheel_r} ${flag*(chasis_w/2-wheel_l/2)} ${-(wheel_r+chasis_h/2)}" rpy="0 0 0"/>
         </joint>

File: xacro/ackermann/imu.xacro (robot description, xacro)
@@ -4,18 +4,18 @@
         <visual>
             <geometry>
-                <box size="0.05 0.05 0.01"/>
+                <box size="${imu_l} ${imu_w} ${imu_h}"/>
             </geometry>
         </visual>
         <collision>
             <geometry>
-                <box size="0.05 0.05 0.01"/>
+                <box size="${imu_l} ${imu_w} ${imu_h}"/>
             </geometry>
         </collision>
-        <xacro:box_inertial_matrix m="0.01" l="0.05" w="0.05" h="0.01"/>
+        <xacro:box_inertial_matrix m="${imu_m}" l="${imu_l}" w="${imu_w}" h="${imu_h}"/>
     </link>
     <joint name="imu2chasis" type="fixed">
         <parent link="chasis"/>
         <child link="imu"/>
-        <origin xyz="0.0 0.0 ${chasis_h/2+0.005}" rpy="0.0 0.0 0.0"/>
+        <origin xyz="${chasis_l/2-wheel_r} 0.0 ${chasis_h/2+imu_h/2}" rpy="0.0 0.0 0.0"/>
     </joint>
     <gazebo reference="imu">

File: xacro/ackermann/lidar.xacro (robot description, xacro)
@@ -12,5 +12,5 @@
         <parent link="chasis"/>
         <child link="lidar"/>
-        <origin xyz="${chasis_l/2-lidar_r} 0.0 ${chasis_h/2+lidar_l/2}" rpy="0.0 0.0 0.0"/>
+        <origin xyz="${chasis_l/2-wheel_r-imu_l/2-lidar_r} 0.0 ${chasis_h/2+lidar_l}" rpy="0.0 0.0 0.0"/>
     </joint>
     <gazebo reference="lidar">

File: xacro/ackermann/racecar.xacro (robot description, xacro)
@@ -13,4 +13,8 @@
     <xacro:property name="lidar_l" value="0.1"/>
     <xacro:property name="lidar_m" value="0.5"/>
+    <xacro:property name="imu_l" value="0.05"/>
+    <xacro:property name="imu_w" value="0.05"/>
+    <xacro:property name="imu_h" value="0.01"/>
+    <xacro:property name="imu_m" value="0.5"/>
     <!-- <xacro:property name="pi" value="3.1415926"/> -->
     <xacro:include filename="$(find test_mycar)/xacro/ackermann/chasis.xacro"/>

File: xacro/tracer/platform.xacro (robot description, xacro)
@@ -24,16 +24,10 @@
         <type>transmission_interface/SimpleTransmission</type>
         <joint name="platform2chasis">
-            <hardwareInterface>hardware_interface/EffortJointInterface</hardwareInterface>
+            <hardwareInterface>PositionJointInterface</hardwareInterface>
         </joint>
         <actuator name="platform2chasis_motor">
             <mechanicalReduction>1.0</mechanicalReduction>
-            <hardwareInterface>hardware_interface/EffortJointInterface</hardwareInterface>
+            <hardwareInterface>PositionJointInterface</hardwareInterface>
         </actuator>
     </transmission>
-    <gazebo>
-        <plugin name="gazebo_ros_control" filename="libgazebo_ros_control.so">
-            <robotNamespace>/tracer</robotNamespace>
-            <robotSimType>gazebo_ros_control</robotSimType>
-        </plugin>
-    </gazebo>
 </robot>

File: xacro/tracer/tracer.xacro (robot description, xacro)
@@ -8,11 +8,11 @@
     </link>
     <xacro:include filename="$(find test_mycar)/xacro/tracer/params.xacro"/>
-    <xacro:include filename="$(find test_mycar)/xacro/tracer/inertia.xacro"/>
+    <xacro:include filename="$(find test_mycar)/xacro/inertia.xacro"/>
+    <!-- <xacro:include filename="$(find test_mycar)/xacro/tracer/platform.xacro"/> -->
     <xacro:include filename="$(find test_mycar)/xacro/tracer/chasis.xacro"/>
-    <xacro:include filename="$(find test_mycar)/xacro/tracer/spheres.xacro"/>
     <xacro:include filename="$(find test_mycar)/xacro/tracer/lidar.xacro"/>
     <!-- <xacro:include filename="$(find test_mycar)/xacro/tracer/camera.xacro"/> -->
     <xacro:include filename="$(find test_mycar)/xacro/tracer/kinect_camera.xacro"/>
-    <xacro:include filename="$(find test_mycar)/xacro/tracer/platform.xacro"/>
+    <xacro:include filename="$(find test_mycar)/xacro/tracer/spheres.xacro"/>
     <xacro:include filename="$(find test_mycar)/xacro/tracer/wheels.xacro"/>
 </robot>

File: xacro/tracer/wheels.xacro (robot description, xacro)
@@ -41,5 +41,5 @@
             <robotNamespace>/</robotNamespace>
             <!-- <publishTf>1</publishTf> -->
-            <!-- <publishWheelJointState>true</publishWheelJointState> -->
+            <publishWheelJointState>true</publishWheelJointState>
             <alwaysOn>true</alwaysOn>
             <updateRate>100.0</updateRate>
@@ -52,9 +52,12 @@
             <wheelTorque>30</wheelTorque>
             <!-- <wheelAcceleration>1.8</wheelAcceleration> -->
-            <commandTopic>cmd_vel</commandTopic> <!-- 运动控制话题 -->
-            <odometryFrame>odom</odometryFrame>
-            <odometryTopic>odom</odometryTopic> <!-- 里程计话题 -->
-            <robotBaseFrame>base_link</robotBaseFrame> <!-- 根坐标系 -->
+            <commandTopic>/cmd_vel</commandTopic> <!-- 运动控制话题 -->
+            <odometryFrame>/odom</odometryFrame>
+            <odometryTopic>/odom</odometryTopic> <!-- 里程计话题 -->
+            <robotBaseFrame>/base_link</robotBaseFrame> <!-- 根坐标系 -->
         </plugin>
+        <!-- <plugin name="gazebo_ros_control" filename="libgazebo_ros_control.so">
+            <robotNamespace>/tracer</robotNamespace>
+        </plugin> -->
     </gazebo>
 </robot>

Commit message: update

File: xacro/ackermann/front_wheels.xacro (robot description, xacro)
@@ -22,6 +22,6 @@
             <parent link="chasis"/>
             <child link="${name}_steering"/>
-            <axis xyz="0 0 1"/>
-            <limit lower="-1.52" upper="1.52" velocity="1.0" effort="1000.0"/>
+            <axis xyz="0 0 -1"/>
+            <limit lower="${-pi/4}" upper="${pi/4}" velocity="4.553" effort="0.5649"/>
             <origin xyz="${chasis_l/2-wheel_r} ${flag*(chasis_w/2-wheel_l/2)} ${-(wheel_r+chasis_h/2)}" rpy="0 0 0"/>
         </joint>
@@ -29,9 +29,9 @@
             <type>transmission_interface/SimpleTransmission</type>
             <joint name="${name}_steering2chasis">
-                <hardwareInterface>hardware_interface/EffortJointInterface</hardwareInterface>
+                <hardwareInterface>hardware_interface/PositionJointInterface</hardwareInterface>
             </joint>
             <actuator name="${name}_steering2chasis_motor">
                 <mechanicalReduction>1.0</mechanicalReduction>
-                <hardwareInterface>hardware_interface/EffortJointInterface</hardwareInterface>
+                <hardwareInterface>hardware_interface/PositionJointInterface</hardwareInterface>
             </actuator>
         </transmission>
@@ -67,4 +67,10 @@
             </actuator>
         </transmission>
+        <gazebo reference="front_${name}_wheel">
+            <mu1 value="100.0"/>
+            <mu2 value="50.0"/>
+            <kp value="1000000.0" />
+            <kd value="10.0" />
+        </gazebo>
     </xacro:macro>
     <xacro:front_wheels_func name="left" flag="1"/>

File: xacro/ackermann/racecar.xacro (robot description, xacro)
@@ -6,11 +6,11 @@
     <xacro:property name="chasis_w" value="0.6"/>
     <xacro:property name="chasis_h" value="0.1"/>
-    <xacro:property name="chasis_m" value="10.0"/>
+    <xacro:property name="chasis_m" value="20.0"/>
     <xacro:property name="wheel_r" value="0.1"/>
     <xacro:property name="wheel_l" value="0.1"/>
-    <xacro:property name="wheel_m" value="2.0"/>
+    <xacro:property name="wheel_m" value="5.0"/>
     <xacro:property name="lidar_r" value="0.1"/>
     <xacro:property name="lidar_l" value="0.1"/>
-    <xacro:property name="lidar_m" value="0.5"/>
+    <xacro:property name="lidar_m" value="1.0"/>
     <xacro:property name="imu_l" value="0.05"/>
     <xacro:property name="imu_w" value="0.05"/>

File: xacro/ackermann/rear_wheels.xacro (robot description, xacro)
@@ -33,4 +33,10 @@
             </actuator>
         </transmission>
+        <gazebo reference="rear_${name}_wheel">
+            <mu1 value="10.0"/>
+            <mu2 value="10.0"/>
+            <kp value="1000000.0" />
+            <kd value="10.0" />
+        </gazebo>
     </xacro:macro>
     <xacro:rear_wheels_func name="left" flag="1"/>
