Commit message: update

File: xacro/ackermann/chasis.xacro (robot description, xacro)
@@ -1,3 +1,21 @@
 <?xml version="1.0"?>
 <robot xmlns:xacro="http://www.ros.org/wiki/xacro" name="racecar">
+    <link name="chasis">
+        <visual >
+            <geometry>
+                <box size="${chasis_l} ${chasis_w} ${chasis_h}"/>
+            </geometry>
+        </visual>
+        <collision>
+            <geometry>
+                <box size="${chasis_l} ${chasis_w} ${chasis_h}"/>
+            </geometry>
+        </collision>
+        <xacro:box_inertial_matrix m="${chasis_m}" l="${chasis_l}" w="${chasis_w}" h="${chasis_h}" />
+    </link>
+    <joint name="chasis2base" type="fixed">
+        <parent link="base_link"/>
+        <child link="chasis"/>
+        <origin xyz="0.0 0.0 ${wheel_r*2+chasis_h/2}" rpy="0.0 0.0 0.0"/>
+    </joint>
 </robot>

File: xacro/ackermann/racecar.xacro (robot description, xacro)
@@ -2,8 +2,28 @@
 <robot xmlns:xacro="http://www.ros.org/wiki/xacro" name="racecar">
     <link name="base_link"/>
-    <xacro:property name="chasis_l" value="0.5"/>
-    <xacro:property name="chasis_w" value="0.3"/>
+    <xacro:include filename="$(find test_mycar)/xacro/inertia.xacro"/>
+    <xacro:property name="chasis_l" value="1.0"/>
+    <xacro:property name="chasis_w" value="0.6"/>
     <xacro:property name="chasis_h" value="0.1"/>
-    <xacro:property name="wheel_r" value="0.2"/>
+    <xacro:property name="chasis_m" value="10.0"/>
+    <xacro:property name="wheel_r" value="0.1"/>
     <xacro:property name="wheel_l" value="0.1"/>
+    <xacro:property name="wheel_m" value="2.0"/>
+    <xacro:property name="lidar_r" value="0.1"/>
+    <xacro:property name="lidar_l" value="0.1"/>
+    <xacro:property name="lidar_m" value="0.5"/>
+    <!-- <xacro:property name="pi" value="3.1415926"/> -->
+    <xacro:include filename="$(find test_mycar)/xacro/ackermann/chasis.xacro"/>
+    <xacro:include filename="$(find test_mycar)/xacro/ackermann/rear_wheels.xacro"/>
+    <xacro:include filename="$(find test_mycar)/xacro/ackermann/front_wheels.xacro"/>
+    <xacro:include filename="$(find test_mycar)/xacro/ackermann/lidar.xacro"/>
+    <xacro:include filename="$(find test_mycar)/xacro/ackermann/imu.xacro"/>
+    <gazebo>
+        <plugin name="gazebo_ros_control" filename="libgazebo_ros_control.so">
+          <robotNamespace>/racecar</robotNamespace>
+          <robotParam>robot_description</robotParam>
+          <robotSimType>gazebo_ros_control/DefaultRobotHWSim</robotSimType>
+          <legacyModeNS>true</legacyModeNS>
+        </plugin>
+    </gazebo>
 </robot>

Commit message: update

File: xacro/ackermann/chasis.xacro (robot description, xacro)
@@ -7,9 +7,9 @@
             </geometry>
         </visual>
-        <collision>
+        <!-- <collision>
             <geometry>
                 <box size="${chasis_l} ${chasis_w} ${chasis_h}"/>
             </geometry>
-        </collision>
+        </collision> -->
         <xacro:box_inertial_matrix m="${chasis_m}" l="${chasis_l}" w="${chasis_w}" h="${chasis_h}" />
     </link>

File: xacro/ackermann/lidar.xacro (robot description, xacro)
@@ -12,10 +12,10 @@
         <parent link="chasis"/>
         <child link="lidar"/>
-        <origin xyz="${chasis_l/2-wheel_r-imu_l/2-lidar_r} 0.0 ${chasis_h/2+lidar_l}" rpy="0.0 0.0 0.0"/>
+        <origin xyz="${chasis_l/2-wheel_r-imu_l/2-lidar_r} 0.0 ${chasis_h*2+lidar_l}" rpy="0.0 0.0 0.0"/>
     </joint>
     <gazebo reference="lidar">
         <sensor type="ray" name="rplidar">
-            <pose>0 0 0 0 0 0</pose>
-            <visualize>false</visualize>
+            <pose>0 0 ${lidar_l} 0 0 0</pose>
+            <visualize>true</visualize>
             <update_rate>20.0</update_rate>
             <ray>

File: xacro/ackermann/racecar.xacro (robot description, xacro)
@@ -2,5 +2,5 @@
 <robot xmlns:xacro="http://www.ros.org/wiki/xacro" name="racecar">
     <link name="base_link"/>
-    <xacro:include filename="$(find test_mycar)/xacro/inertia.xacro"/>
+    <xacro:include filename="$(find my_gazebo_sim)/xacro/inertia.xacro"/>
     <xacro:property name="chasis_l" value="1.0"/>
     <xacro:property name="chasis_w" value="0.6"/>
@@ -18,9 +18,9 @@
     <xacro:property name="imu_m" value="0.5"/>
     <!-- <xacro:property name="pi" value="3.1415926"/> -->
-    <xacro:include filename="$(find test_mycar)/xacro/ackermann/chasis.xacro"/>
-    <xacro:include filename="$(find test_mycar)/xacro/ackermann/rear_wheels.xacro"/>
-    <xacro:include filename="$(find test_mycar)/xacro/ackermann/front_wheels.xacro"/>
-    <xacro:include filename="$(find test_mycar)/xacro/ackermann/lidar.xacro"/>
-    <xacro:include filename="$(find test_mycar)/xacro/ackermann/imu.xacro"/>
+    <xacro:include filename="$(find my_gazebo_sim)/xacro/ackermann/chasis.xacro"/>
+    <xacro:include filename="$(find my_gazebo_sim)/xacro/ackermann/rear_wheels.xacro"/>
+    <xacro:include filename="$(find my_gazebo_sim)/xacro/ackermann/front_wheels.xacro"/>
+    <xacro:include filename="$(find my_gazebo_sim)/xacro/ackermann/lidar.xacro"/>
+    <xacro:include filename="$(find my_gazebo_sim)/xacro/ackermann/imu.xacro"/>
     <gazebo>
         <plugin name="gazebo_ros_control" filename="libgazebo_ros_control.so">

File: xacro/tracer/tracer.xacro (robot description, xacro)
@@ -27,12 +27,12 @@
         </visual>
     </link>
-    <xacro:include filename="$(find test_mycar)/xacro/inertia.xacro"/>
-    <xacro:include filename="$(find test_mycar)/xacro/tracer/platform.xacro"/>
-    <xacro:include filename="$(find test_mycar)/xacro/tracer/chasis.xacro"/>
-    <xacro:include filename="$(find test_mycar)/xacro/tracer/lidar.xacro"/>
-    <!-- <xacro:include filename="$(find test_mycar)/xacro/tracer/camera.xacro"/> -->
-    <xacro:include filename="$(find test_mycar)/xacro/tracer/kinect_camera.xacro"/>
-    <xacro:include filename="$(find test_mycar)/xacro/tracer/spheres.xacro"/>
-    <xacro:include filename="$(find test_mycar)/xacro/tracer/wheels.xacro"/>
-    <xacro:include filename="$(find test_mycar)/xacro/tracer/imu.xacro"/>
+    <xacro:include filename="$(find my_gazebo_sim)/xacro/inertia.xacro"/>
+    <xacro:include filename="$(find my_gazebo_sim)/xacro/tracer/platform.xacro"/>
+    <xacro:include filename="$(find my_gazebo_sim)/xacro/tracer/chasis.xacro"/>
+    <xacro:include filename="$(find my_gazebo_sim)/xacro/tracer/lidar.xacro"/>
+    <!-- <xacro:include filename="$(find my_gazebo_sim)/xacro/tracer/camera.xacro"/> -->
+    <xacro:include filename="$(find my_gazebo_sim)/xacro/tracer/kinect_camera.xacro"/>
+    <xacro:include filename="$(find my_gazebo_sim)/xacro/tracer/spheres.xacro"/>
+    <xacro:include filename="$(find my_gazebo_sim)/xacro/tracer/wheels.xacro"/>
+    <xacro:include filename="$(find my_gazebo_sim)/xacro/tracer/imu.xacro"/>
 </robot>
